File: PCB/uLED_v1.sch (EAGLE design)
At the start: 6 parts, among them IC1 ATSAMD21E, Q1 reset, Q2 reset

Commit message: save from my battery
Parts:
- added R1, R2, R3: .330, SparkFun-Resistors:0.27OHM-0603-1/10W-1%
Connections:
- removed net AIN[1]: D1.RED, IC1.PA03/EINT3/VREFA/AIN1
- removed net AIN[4]: IC1.PA04/EINT4/VREFB/AIN4/SERCOM0.0
- removed net AIN[5]: IC1.PA05/EINT5/AIN5/SERCOM0.1
- removed net TIM3/WO[1]: IC1.PA19/I3/SERCOM1+3.3/I2SD0
- new net N$1: D1.RED, R1.2
- new net TIM3/WO[1]/AIN[1]: IC1.PA03/EINT3/VREFA/AIN1, IC1.PA19/I3/SERCOM1+3.3/I2SD0, R1.1
- net N$2: now also R3.2
- net N$3: now also R2.2
- net TIM4/WO[1]: now also R2.1
- net TIM5/WO[0]: now also R3.1
Other:
- note removed: "TODO: Attach AIN and TIMX to each of the diodes"
Changed lines of the file:
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@@
 <?xml version="1.0" encoding="utf-8"?>
 <!DOCTYPE eagle SYSTEM "eagle.dtd">
-<eagle version="9.2.1">
+<eagle version="9.2.0">
 <drawing>
 <settings>
@@
 <part name="Q2" library="microbuilder" deviceset="SWITCH_TACT_SMT" device="4.6X2.8" value="reset"/>
 <part name="D1" library="SparkFun-LED" library_urn="urn:adsk.eagle:library:529" deviceset="LED-RGB-CA" device="CLEAR" package3d_urn="urn:adsk.eagle:package:39368/1" value="CLEAR"/>
+<part name="R1" library="SparkFun-Resistors" library_urn="urn:adsk.eagle:library:532" deviceset="0.27OHM" device="-0603-1/10W-1%" package3d_urn="urn:adsk.eagle:package:39650/1" value=".330"/>
+<part name="R2" library="SparkFun-Resistors" library_urn="urn:adsk.eagle:library:532" deviceset="0.27OHM" device="-0603-1/10W-1%" package3d_urn="urn:adsk.eagle:package:39650/1" value=".330"/>
+<part name="R3" library="SparkFun-Resistors" library_urn="urn:adsk.eagle:library:532" deviceset="0.27OHM" device="-0603-1/10W-1%" package3d_urn="urn:adsk.eagle:package:39650/1" value=".330"/>
 </parts>
 <sheets>
 <sheet>
 <plain>
-<text x="184.15" y="41.91" size="1.778" layer="91">TODO: Attach AIN and TIMX to each of the diodes</text>
 <text x="191.77" y="38.1" size="1.778" layer="91">Import parts</text>
 </plain>
 <instances>
-<instance part="IC1" gate="G$1" x="87.63" y="43.18" smashed="yes">
+<instance part="IC1" gate="G$1" x="87.63" y="43.18">
 <attribute name="NAME" x="52.07" y="0" size="1.778" layer="95"/>
 <attribute name="VALUE" x="57.15" y="88.9" size="1.778" layer="96"/>
 </instance>
-<instance part="GND5" gate="1" x="8.89" y="86.36" smashed="yes">
+<instance part="GND5" gate="1" x="8.89" y="86.36">
 <attribute name="VALUE" x="6.35" y="83.82" size="1.778" layer="96"/>
 </instance>
-<instance part="TP1" gate="G$1" x="31.75" y="91.44" smashed="yes" rot="MR0">
+<instance part="TP1" gate="G$1" x="31.75" y="91.44" rot="MR0">
 <attribute name="NAME" x="33.02" y="92.71" size="1.778" layer="95" rot="MR0"/>
 <attribute name="TP_SIGNAL_NAME" x="30.48" y="90.17" size="1.778" layer="97" rot="MR0"/>
 </instance>
-<instance part="Q1" gate="G$1" x="19.05" y="91.44" smashed="yes" rot="MR0">
+<instance part="Q1" gate="G$1" x="19.05" y="91.44" rot="MR0">
 <attribute name="NAME" x="21.59" y="97.79" size="1.27" layer="95" rot="MR0"/>
 <attribute name="VALUE" x="21.59" y="86.36" size="1.27" layer="96" rot="MR0"/>
 </instance>
-<instance part="U$11" gate="G$1" x="27.94" y="78.74" smashed="yes">
+<instance part="U$11" gate="G$1" x="27.94" y="78.74">
 <attribute name="VALUE" x="26.416" y="79.756" size="1.27" layer="96"/>
 </instance>
-<instance part="C3" gate="G$1" x="36.83" y="60.96" smashed="yes">
+<instance part="C3" gate="G$1" x="36.83" y="60.96">
 <attribute name="NAME" x="34.54" y="62.21" size="1.27" layer="95" font="vector" rot="R90" align="center"/>
 <attribute name="VALUE" x="39.13" y="62.21" size="1.27" layer="96" font="vector" rot="R90" align="center"/>
 </instance>
-<instance part="GND1" gate="1" x="38.1" y="0" smashed="yes">
+<instance part="GND1" gate="1" x="38.1" y="0">
 <attribute name="VALUE" x="38.1" y="-0.254" size="1.778" layer="96" align="top-center"/>
 </instance>
-<instance part="GND2" gate="1" x="36.83" y="55.88" smashed="yes">
+<instance part="GND2" gate="1" x="36.83" y="55.88">
 <attribute name="VALUE" x="36.83" y="55.626" size="1.778" layer="96" align="top-center"/>
 </instance>
-<instance part="GND3" gate="1" x="161.29" y="40.64" smashed="yes" rot="MR0">
+<instance part="GND3" gate="1" x="161.29" y="40.64" rot="MR0">
 <attribute name="VALUE" x="163.83" y="38.1" size="1.778" layer="96" rot="MR0"/>
 </instance>
-<instance part="Q2" gate="G$1" x="152.4" y="45.72" smashed="yes">
+<instance part="Q2" gate="G$1" x="152.4" y="45.72">
 <attribute name="NAME" x="149.86" y="52.07" size="1.27" layer="95"/>
 </instance>
-<instance part="D1" gate="G$1" x="210.82" y="86.36" smashed="yes" rot="R90">
+<instance part="D1" gate="G$1" x="210.82" y="86.36" rot="R90">
 <attribute name="NAME" x="205.4225" y="78.74" size="1.778" layer="95" font="vector" rot="R90"/>
 <attribute name="VALUE" x="216.2175" y="78.74" size="1.778" layer="95" font="vector" rot="R90" align="top-left"/>
+</instance>
+<instance part="R1" gate="G$1" x="203.2" y="71.12" rot="R90">
+<attribute name="NAME" x="201.676" y="71.12" size="1.778" layer="95" font="vector" rot="R90" align="bottom-center"/>
+<attribute name="VALUE" x="204.724" y="71.12" size="1.778" layer="96" font="vector" rot="R90" align="top-center"/>
+</instance>
+<instance part="R2" gate="G$1" x="210.82" y="66.04" rot="R90">
+<attribute name="NAME" x="209.296" y="66.04" size="1.778" layer="95" font="vector" rot="R90" align="bottom-center"/>
+<attribute name="VALUE" x="212.344" y="66.04" size="1.778" layer="96" font="vector" rot="R90" align="top-center"/>
+</instance>
+<instance part="R3" gate="G$1" x="218.44" y="71.12" rot="R90">
+<attribute name="NAME" x="216.916" y="71.12" size="1.778" layer="95" font="vector" rot="R90" align="bottom-center"/>
+<attribute name="VALUE" x="219.964" y="71.12" size="1.778" layer="96" font="vector" rot="R90" align="top-center"/>
 </instance>
 </instances>
@@
 </segment>
 </net>
-<net name="AIN[1]" class="0">
-<segment>
-<pinref part="IC1" gate="G$1" pin="PA03/EINT3/VREFA/AIN1"/>
-<wire x1="123.19" y1="76.2" x2="133.35" y2="76.2" width="0.1524" layer="91"/>
-<label x="125.73" y="76.2" size="1.778" layer="95"/>
-</segment>
-<segment>
-<pinref part="D1" gate="G$1" pin="RED"/>
-<wire x1="208.28" y1="76.2" x2="208.28" y2="74.93" width="0.1524" layer="91"/>
-<wire x1="208.28" y1="74.93" x2="204.47" y2="74.93" width="0.1524" layer="91"/>
-<wire x1="204.47" y1="74.93" x2="204.47" y2="68.58" width="0.1524" layer="91"/>
-<junction x="208.28" y="74.93"/>
-<wire x1="208.28" y1="74.93" x2="208.28" y2="68.58" width="0.1524" layer="91"/>
-</segment>
-</net>
-<net name="AIN[4]" class="0">
-<segment>
-<pinref part="IC1" gate="G$1" pin="PA04/EINT4/VREFB/AIN4/SERCOM0.0"/>
-<wire x1="123.19" y1="73.66" x2="133.35" y2="73.66" width="0.1524" layer="91"/>
-<label x="125.73" y="73.66" size="1.778" layer="95"/>
-</segment>
-</net>
-<net name="AIN[5]" class="0">
-<segment>
-<pinref part="IC1" gate="G$1" pin="PA05/EINT5/AIN5/SERCOM0.1"/>
-<wire x1="123.19" y1="71.12" x2="133.35" y2="71.12" width="0.1524" layer="91"/>
-<label x="125.73" y="71.12" size="1.778" layer="95"/>
-</segment>
-</net>
-<net name="TIM3/WO[1]" class="0">
-<segment>
-<pinref part="IC1" gate="G$1" pin="PA19/I3/SERCOM1+3.3/I2SD0"/>
-<wire x1="123.19" y1="30.48" x2="133.35" y2="30.48" width="0.1524" layer="91"/>
-<label x="125.73" y="30.48" size="1.778" layer="95"/>
-</segment>
-</net>
 <net name="TIM4/WO[1]" class="0">
 <segment>
@@
 <label x="125.73" y="17.78" size="1.778" layer="95"/>
 </segment>
+<segment>
+<pinref part="R2" gate="G$1" pin="1"/>
+<wire x1="210.82" y1="60.96" x2="210.82" y2="55.88" width="0.1524" layer="91"/>
+<label x="210.82" y="48.26" size="1.778" layer="95" rot="R90"/>
+</segment>
 </net>
 <net name="TIM5/WO[0]" class="0">
@@
 <wire x1="123.19" y1="15.24" x2="133.35" y2="15.24" width="0.1524" layer="91"/>
 <label x="125.73" y="15.24" size="1.778" layer="95"/>
+</segment>
+<segment>
+<pinref part="R3" gate="G$1" pin="1"/>
+<wire x1="218.44" y1="66.04" x2="218.44" y2="55.88" width="0.1524" layer="91"/>
+<label x="215.9" y="60.96" size="1.778" layer="95" rot="R270"/>
 </segment>
 </net>
@@
 <segment>
 <pinref part="D1" gate="G$1" pin="GRN"/>
-<wire x1="213.36" y1="76.2" x2="213.36" y2="74.93" width="0.1524" layer="91"/>
-<wire x1="213.36" y1="74.93" x2="213.36" y2="68.58" width="0.1524" layer="91"/>
-<wire x1="213.36" y1="74.93" x2="217.17" y2="74.93" width="0.1524" layer="91"/>
-<wire x1="217.17" y1="74.93" x2="217.17" y2="68.58" width="0.1524" layer="91"/>
-<junction x="213.36" y="74.93"/>
+<wire x1="213.36" y1="76.2" x2="218.44" y2="76.2" width="0.1524" layer="91"/>
+<pinref part="R3" gate="G$1" pin="2"/>
 </segment>
 </net>
@@
 <segment>
 <pinref part="D1" gate="G$1" pin="BLU"/>
-<wire x1="210.82" y1="76.2" x2="210.82" y2="63.5" width="0.1524" layer="91"/>
-<wire x1="210.82" y1="63.5" x2="208.28" y2="63.5" width="0.1524" layer="91"/>
-<wire x1="208.28" y1="63.5" x2="208.28" y2="58.42" width="0.1524" layer="91"/>
-<wire x1="210.82" y1="63.5" x2="213.36" y2="63.5" width="0.1524" layer="91"/>
-<junction x="210.82" y="63.5"/>
-<wire x1="213.36" y1="63.5" x2="213.36" y2="58.42" width="0.1524" layer="91"/>
-</segment>
-</net>
+<wire x1="210.82" y1="76.2" x2="210.82" y2="71.12" width="0.1524" layer="91"/>
+<pinref part="R2" gate="G$1" pin="2"/>
+</segment>
+</net>
+<net name="TIM3/WO[1]/AIN[1]" class="0">
+<segment>
+<pinref part="IC1" gate="G$1" pin="PA03/EINT3/VREFA/AIN1"/>
+<wire x1="123.19" y1="76.2" x2="133.35" y2="76.2" width="0.1524" layer="91"/>
+<label x="125.73" y="76.2" size="1.778" layer="95"/>
+</segment>
+<segment>
+<pinref part="IC1" gate="G$1" pin="PA19/I3/SERCOM1+3.3/I2SD0"/>
+<wire x1="123.19" y1="30.48" x2="133.35" y2="30.48" width="0.1524" layer="91"/>
+<label x="125.73" y="30.48" size="1.778" layer="95"/>
+</segment>
+<segment>
+<pinref part="R1" gate="G$1" pin="1"/>
+<wire x1="203.2" y1="66.04" x2="203.2" y2="55.88" width="0.1524" layer="91"/>
+<label x="203.2" y="48.26" size="1.778" layer="95" rot="R90"/>
+</segment>
+</net>
+<net name="N$1" class="0">
+<segment>
+<pinref part="D1" gate="G$1" pin="RED"/>
+<pinref part="R1" gate="G$1" pin="2"/>
+<wire x1="203.2" y1="76.2" x2="208.28" y2="76.2" width="0.1524" layer="91"/>
+</segment>
+</net>

Commit message: Updated PCB
Parts:
- removed TP1: TPTP16R, testpad:TPTP16R
- added BT1: (no value), SparkFun-Batteries:BATTERY-12MM_PTH
- CONTROL, RESET: value reset -> (none)
- R1, R2, R3: value .330 -> 330Ω
- renumbered Q1 to RESET, Q2 to CONTROL
Connections:
- net A renamed ANODE
- removed net 3.3V: IC1.VDDA, IC1.VDDIN
- removed net SERCOM0/PAD[0]: IC1.PA08/I2C/AIN16/SERCOM0+2.0/I2SD1
- removed net SERCOM0/PAD[1]: IC1.PA09/I2C/I9/AIN17/SERCOM0+2.1/I2SMC
- removed net SERCOM0/PAD[2]: IC1.PA10/I10/AIN18/SERCOM0+2.2/I2SCK
- removed net SERCOM0/PAD[3]: IC1.PA11/I11/AIN19/SERCOM0+2.3/I2SF0
- removed net TIM3/WO[1]/AIN[1]: IC1.PA03/EINT3/VREFA/AIN1, IC1.PA19/I3/SERCOM1+3.3/I2SD0, R1.1
- removed net TIM4/WO[1]: IC1.PA23/I2C/I7/SERCOM3+5.1/SOF, R2.1
- removed net TIM5/WO[0]: IC1.PA24/I12/SERCOM3+5.2/D-, R3.1
- new net BLUEOUT: IC1.PA10/I10/AIN18/SERCOM0+2.2/I2SCK, R3.1
- new net GREENOUT: IC1.PA09/I2C/I9/AIN17/SERCOM0+2.1/I2SMC, R2.1
- new net N$4: BT1.+, IC1.VDDA, IC1.VDDIN
- new net REDOUT: IC1.PA08/I2C/AIN16/SERCOM0+2.0/I2SD1, R1.1
- new net SERCOM_1+3.0: IC1.PA16/I2C/I0/SERCOM1+3.0
- new net SERCOM_1+3.1: IC1.PA17/I2C/I1/SERCOM1+3.1
- net GND: now also BT1.-
- net RESETN: no longer TP1.TP

Commit message: PBG in progress
Parts:
- removed CONTROL: (no value), microbuilder:SWITCH_TACT_SMT4.6X2.8
- added C1, C8: 10uF, microbuilder:CAP_CERAMIC0805-NOOUTLINE
- added C2: 1uF, microbuilder:CAP_CERAMIC0603_NO
- added CTRL: (no value), microbuilder:SWITCH_TACT_SMT4.6X2.8
- added J1: (no value), SparkFun-Connectors:CONN_04
- added J2: 455-1750-1-ND, SparkFun-Connectors:CONN_03
- added LED1: AP102-2020, microbuilder:APA1022020
- added SW1: EG1218, microbuilder:SWITCH_DPDTEG1390
- added U1: AP2112K-3.3, microbuilder:VREG_SOT23-5
- D1: value CLEAR -> SCHOTTKY; device SparkFun-LED:LED-RGB-CACLEAR -> adafruit:DIODE_SOD-123FL
Connections:
- removed net N$4: BT1.+, IC1.VDDA, IC1.VDDIN
- new net 3.3V: C2.1, C8.1, IC1.VDDA, IC1.VDDIN, LED1.VDD, U1.OUT
- new net VBAT: BT1.+, D1.A
- new net VHIGH: D1.C, SW1.O2
- new net VOUT: C1.1, SW1.P2, U1.EN, U1.IN
- net ANODE: now also IC1.PA07/I7/AIN7/SERCOM0.3/I2SD0, J1.2; no longer D1.A, IC1.PA22/I2C/I6/SERCOM3+5.0
- net BUTTON: now also CTRL.P, CTRL.P1, IC1.PA22/I2C/I6/SERCOM3+5.0; no longer CONTROL.P, CONTROL.P1, IC1.PA14/I14/SERCOM2+4.2
- net GND: now also C1.2, C2.2, C8.2, CTRL.S, CTRL.S1, LED1.GND, U1.GND; no longer CONTROL.S, CONTROL.S1
- net N$1: now also J1.1; no longer D1.RED
- net N$2: now also J1.4; no longer D1.GRN
- net N$3: now also J1.3; no longer D1.BLU
- net RESETN: now also J2.1
- net SCDIO: now also J2.3
- net SWCLK: now also J2.2
Other:
- note removed: "Import parts"
- moved on the sheet: BT1, C3, R1, R2, R3

Commit message: Updating board again
Parts:
- removed BT1: (no value), SparkFun-Batteries:BATTERY-12MM_PTH
- added BT2: (no value), SparkFun-Batteries:BATTERY-20MM_SMD
Connections:
- new net LEDCI: IC1.PA06/EINT6/AIN6/SERCOM0.2, LED1.CKI
- new net LEDDI: IC1.PA07/I7/AIN7/SERCOM0.3/I2SD0, LED1.DI
- net ANODE: now also IC1.PA11/I11/AIN19/SERCOM0+2.3/I2SF0; no longer IC1.PA07/I7/AIN7/SERCOM0.3/I2SD0
- net GND: now also BT2.-; no longer BT1.-
- net VBAT: now also BT2.+; no longer BT1.+
Other:
- moved on the sheet: LED1, SW1
Changed lines of the file:
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@@
 <part name="R2" library="SparkFun-Resistors" library_urn="urn:adsk.eagle:library:532" deviceset="0.27OHM" device="-0603-1/10W-1%" package3d_urn="urn:adsk.eagle:package:39650/1" value="330Ω"/>
 <part name="R3" library="SparkFun-Resistors" library_urn="urn:adsk.eagle:library:532" deviceset="0.27OHM" device="-0603-1/10W-1%" package3d_urn="urn:adsk.eagle:package:39650/1" value="330Ω"/>
-<part name="BT1" library="SparkFun-Batteries" deviceset="BATTERY" device="-12MM_PTH"/>
 <part name="J1" library="SparkFun-Connectors" deviceset="CONN_04" device=""/>
 <part name="GND12" library="supply1" deviceset="GND" device=""/>
@@
 <part name="GND8" library="supply1" deviceset="GND" device=""/>
 <part name="J2" library="SparkFun-Connectors" deviceset="CONN_03" device="" value="455-1750-1-ND"/>
+<part name="BT2" library="SparkFun-Batteries" deviceset="BATTERY" device="-20MM_SMD"/>
 </parts>
 <sheets>
@@
 <attribute name="VALUE" x="232.664" y="71.12" size="1.778" layer="96" font="vector" rot="R90" align="top-center"/>
 </instance>
-<instance part="BT1" gate="G$1" x="20.32" y="-30.48" rot="R270">
-<attribute name="NAME" x="24.638" y="-30.48" size="1.778" layer="95" font="vector" rot="R270" align="bottom-center"/>
-<attribute name="VALUE" x="16.002" y="-30.48" size="1.778" layer="96" font="vector" rot="R270" align="top-center"/>
-</instance>
 <instance part="J1" gate="G$1" x="195.58" y="88.9">
 <attribute name="VALUE" x="190.5" y="81.534" size="1.778" layer="96" font="vector"/>
@@
 <attribute name="VALUE" x="63.5" y="-71.12" size="1.778" layer="96" rot="MR0"/>
 </instance>
-<instance part="SW1" gate="G$1" x="45.72" y="-63.5" rot="MR0">
-<attribute name="VALUE" x="50.8" y="-74.93" size="1.27" layer="96" rot="MR0"/>
-<attribute name="NAME" x="50.165" y="-54.61" size="1.27" layer="95" rot="MR0"/>
+<instance part="SW1" gate="G$1" x="45.72" y="-63.5" rot="R180">
+<attribute name="VALUE" x="50.8" y="-52.07" size="1.27" layer="96" rot="R180"/>
+<attribute name="NAME" x="50.165" y="-72.39" size="1.27" layer="95" rot="R180"/>
 </instance>
 <instance part="U$12" gate="G$1" x="104.14" y="-38.1">
@@
 <attribute name="VALUE" x="22.86" y="-43.18" size="1.778" layer="96" rot="MR0"/>
 </instance>
-<instance part="LED1" gate="G$1" x="200.66" y="2.54">
-<attribute name="NAME" x="190.5" y="13.716" size="1.27" layer="95"/>
-<attribute name="VALUE" x="190.5" y="-10.16" size="1.27" layer="96"/>
+<instance part="LED1" gate="G$1" x="200.66" y="5.08">
+<attribute name="NAME" x="190.5" y="16.256" size="1.27" layer="95"/>
+<attribute name="VALUE" x="190.5" y="-7.62" size="1.27" layer="96"/>
 </instance>
 <instance part="U$13" gate="G$1" x="205.74" y="22.86">
@@
 <attribute name="VALUE" x="157.48" y="-10.414" size="1.778" layer="96" font="vector" rot="R180"/>
 <attribute name="NAME" x="157.48" y="-23.368" size="1.778" layer="95" font="vector" rot="R180"/>
+</instance>
+<instance part="BT2" gate="G$1" x="20.32" y="-30.48" rot="R270">
+<attribute name="NAME" x="24.638" y="-30.48" size="1.778" layer="95" font="vector" rot="R270" align="bottom-center"/>
+<attribute name="VALUE" x="16.002" y="-30.48" size="1.778" layer="96" font="vector" rot="R270" align="top-center"/>
 </instance>
 </instances>
@@
 <segment>
 <pinref part="GND7" gate="1" pin="GND"/>
-<pinref part="BT1" gate="G$1" pin="-"/>
 <wire x1="20.32" y1="-38.1" x2="20.32" y2="-35.56" width="0.1524" layer="91"/>
+<pinref part="BT2" gate="G$1" pin="-"/>
 </segment>
 <segment>
 <pinref part="LED1" gate="G$1" pin="GND"/>
 <pinref part="GND8" gate="1" pin="GND"/>
-<wire x1="200.66" y1="-10.16" x2="200.66" y2="-15.24" width="0.1524" layer="91"/>
+<wire x1="200.66" y1="-7.62" x2="200.66" y2="-15.24" width="0.1524" layer="91"/>
 </segment>
 </net>
@@
 <net name="ANODE" class="0">
 <segment>
-<label x="125.73" y="66.04" size="1.778" layer="95"/>
-<pinref part="IC1" gate="G$1" pin="PA07/I7/AIN7/SERCOM0.3/I2SD0"/>
-<wire x1="123.19" y1="66.04" x2="133.35" y2="66.04" width="0.1524" layer="91"/>
+<label x="125.73" y="53.34" size="1.778" layer="95"/>
+<pinref part="IC1" gate="G$1" pin="PA11/I11/AIN19/SERCOM0+2.3/I2SF0"/>
+<wire x1="123.19" y1="53.34" x2="133.35" y2="53.34" width="0.1524" layer="91"/>
 </segment>
 <segment>
@@
 </segment>
 <segment>
-<pinref part="BT1" gate="G$1" pin="+"/>
 <pinref part="U$2" gate="G$1" pin="VBAT"/>
 <wire x1="20.32" y1="-25.4" x2="20.32" y2="-22.86" width="0.1524" layer="91"/>
+<pinref part="BT2" gate="G$1" pin="+"/>
 </segment>
 </net>
@@
 <pinref part="LED1" gate="G$1" pin="VDD"/>
 <pinref part="U$13" gate="G$1" pin="3.3V"/>
-<wire x1="205.74" y1="15.24" x2="205.74" y2="20.32" width="0.1524" layer="91"/>
+<wire x1="205.74" y1="17.78" x2="205.74" y2="20.32" width="0.1524" layer="91"/>
 </segment>
 </net>
@@
 <wire x1="33.02" y1="-48.26" x2="40.64" y2="-48.26" width="0.1524" layer="91"/>
 <pinref part="SW1" gate="G$1" pin="O2"/>
-<wire x1="40.64" y1="-48.26" x2="40.64" y2="-66.04" width="0.1524" layer="91"/>
-<wire x1="40.64" y1="-66.04" x2="43.18" y2="-66.04" width="0.1524" layer="91"/>
+<wire x1="40.64" y1="-48.26" x2="40.64" y2="-60.96" width="0.1524" layer="91"/>
+<wire x1="40.64" y1="-60.96" x2="43.18" y2="-60.96" width="0.1524" layer="91"/>
 </segment>
 </net>
@@
 <label x="50.8" y="-48.26" size="1.778" layer="95"/>
 <pinref part="SW1" gate="G$1" pin="P2"/>
-<wire x1="50.8" y1="-68.58" x2="53.34" y2="-68.58" width="0.1524" layer="91"/>
-<wire x1="53.34" y1="-68.58" x2="53.34" y2="-48.26" width="0.1524" layer="91"/>
-</segment>
-</net>
+<wire x1="53.34" y1="-58.42" x2="53.34" y2="-48.26" width="0.1524" layer="91"/>
+<wire x1="50.8" y1="-58.42" x2="53.34" y2="-58.42" width="0.1524" layer="91"/>
+</segment>
+</net>
+<net name="LEDDI" class="0">
+<segment>
+<pinref part="LED1" gate="G$1" pin="DI"/>
+<wire x1="187.96" y1="0" x2="180.34" y2="0" width="0.1524" layer="91"/>
+<label x="180.34" y="0" size="1.778" layer="95"/>
+</segment>
+<segment>
+<pinref part="IC1" gate="G$1" pin="PA07/I7/AIN7/SERCOM0.3/I2SD0"/>
+<wire x1="123.19" y1="66.04" x2="132.08" y2="66.04" width="0.1524" layer="91"/>
+<label x="125.73" y="66.04" size="1.778" layer="95"/>
+</segment>
+</net>
+<net name="LEDCI" class="0">
+<segment>
+<pinref part="LED1" gate="G$1" pin="CKI"/>
+<wire x1="187.96" y1="-2.54" x2="180.34" y2="-2.54" width="0.1524" layer="91"/>
+<label x="180.34" y="-2.54" size="1.778" layer="95"/>
+</segment>
+<segment>
+<pinref part="IC1" gate="G$1" pin="PA06/EINT6/AIN6/SERCOM0.2"/>
+<wire x1="123.19" y1="68.58" x2="132.08" y2="68.58" width="0.1524" layer="91"/>
+<label x="125.73" y="68.58" size="1.778" layer="95"/>
+</segment>
+</net>

Commit message: yet another pcb
Parts:
- removed BT2: (no value), SparkFun-Batteries:BATTERY-20MM_SMD
- added U$3: 20MM_BATTERY, mikes:20MM_BATTERY
Connections:
- net GND: now also U$3.-; no longer BT2.-
- net VBAT: now also U$3.+2; no longer BT2.+
- net VHIGH: now also SW1.O1; no longer SW1.O2
- net VOUT: now also SW1.P1; no longer SW1.P2
Changed lines of the file:
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@@
 <part name="GND8" library="supply1" deviceset="GND" device=""/>
 <part name="J2" library="SparkFun-Connectors" deviceset="CONN_03" device="" value="455-1750-1-ND"/>
-<part name="BT2" library="SparkFun-Batteries" deviceset="BATTERY" device="-20MM_SMD"/>
+<part name="U$3" library="mikes" deviceset="20MM_BATTERY" device=""/>
 </parts>
 <sheets>
@@
 <attribute name="NAME" x="157.48" y="-23.368" size="1.778" layer="95" font="vector" rot="R180"/>
 </instance>
-<instance part="BT2" gate="G$1" x="20.32" y="-30.48" rot="R270">
+<instance part="U$3" gate="G$1" x="20.32" y="-30.48" rot="R270">
 <attribute name="NAME" x="24.638" y="-30.48" size="1.778" layer="95" font="vector" rot="R270" align="bottom-center"/>
 <attribute name="VALUE" x="16.002" y="-30.48" size="1.778" layer="96" font="vector" rot="R270" align="top-center"/>
@@
 <pinref part="GND7" gate="1" pin="GND"/>
 <wire x1="20.32" y1="-38.1" x2="20.32" y2="-35.56" width="0.1524" layer="91"/>
-<pinref part="BT2" gate="G$1" pin="-"/>
+<pinref part="U$3" gate="G$1" pin="-"/>
 </segment>
 <segment>
@@
 <segment>
 <pinref part="U$2" gate="G$1" pin="VBAT"/>
-<wire x1="20.32" y1="-25.4" x2="20.32" y2="-22.86" width="0.1524" layer="91"/>
-<pinref part="BT2" gate="G$1" pin="+"/>
+<pinref part="U$3" gate="G$1" pin="+2"/>
+<wire x1="22.86" y1="-25.4" x2="22.86" y2="-22.86" width="0.1524" layer="91"/>
+<wire x1="22.86" y1="-22.86" x2="20.32" y2="-22.86" width="0.1524" layer="91"/>
 </segment>
 </net>
@@
 <wire x1="33.02" y1="-40.64" x2="33.02" y2="-48.26" width="0.1524" layer="91"/>
 <wire x1="33.02" y1="-48.26" x2="40.64" y2="-48.26" width="0.1524" layer="91"/>
-<pinref part="SW1" gate="G$1" pin="O2"/>
-<wire x1="40.64" y1="-48.26" x2="40.64" y2="-60.96" width="0.1524" layer="91"/>
-<wire x1="40.64" y1="-60.96" x2="43.18" y2="-60.96" width="0.1524" layer="91"/>
+<pinref part="SW1" gate="G$1" pin="O1"/>
+<wire x1="43.18" y1="-71.12" x2="40.64" y2="-71.12" width="0.1524" layer="91"/>
+<wire x1="40.64" y1="-71.12" x2="40.64" y2="-48.26" width="0.1524" layer="91"/>
 </segment>
 </net>
@@
 <junction x="60.96" y="-48.26"/>
 <label x="50.8" y="-48.26" size="1.778" layer="95"/>
-<pinref part="SW1" gate="G$1" pin="P2"/>
-<wire x1="53.34" y1="-58.42" x2="53.34" y2="-48.26" width="0.1524" layer="91"/>
-<wire x1="50.8" y1="-58.42" x2="53.34" y2="-58.42" width="0.1524" layer="91"/>
-</segment>
-</net>
+<pinref part="SW1" gate="G$1" pin="P1"/>
+<wire x1="50.8" y1="-68.58" x2="53.34" y2="-68.58" width="0.1524" layer="91"/>
+<wire x1="53.34" y1="-68.58" x2="53.34" y2="-48.26" width="0.1524" layer="91"/>
+</segment>
+</net>
